File: Testing.sch (KiCad schematic (older format))
At the start: 18 parts, among them J1 In, J2 LED, J3 Gnd, J4 Jack-DC, J5 Out, J6 In Sleeve, J7 Out Sleeve, Q1 BS170

Commit message: cleaning, add README
Parts:
- D1: footprint Diode_THT:D_DO-41_SOD81_P10.16mm_Horizontal -> Diode_THT:D_DO-41_SOD81_P7.62mm_Horizontal
Other:
- moved on the sheet: C1, C2, D1, D2, J1, J2, J3, J4, J5, J6, J7, Q1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
