File: Testing.sch (KiCad schematic (older format))
At the start: 18 parts, among them J1 In, J2 LED, J3 Gnd, J4 Jack-DC, J5 Out, J6 In Sleeve, J7 Out Sleeve, Q1 BS170

Commit message: pcb layout: move some things around
This mostly involved swapping the transistor with the output coupling
capacitor so that the amplifier and feedback was on the left, and the
output stages were on the right.  I also rotated one resistor so the
nets were closer to each other, and swapped a few of the traces to other
layers of the PCB so that they could be shorter as well.

Overall, the result is pretty much just shorter traces and beefier
power-rail-fill in spots.
Parts:
- D1: footprint Diode_THT:D_DO-41_SOD81_P10.16mm_Horizontal -> Diode_THT:D_DO-41_SOD81_P7.62mm_Horizontal
Changed lines of the file:
@@
 F 0 "D1" V 5704 4229 50  0000 L CNN
 F 1 "1N47xxA" V 5795 4229 50  0000 L CNN
-F 2 "Diode_THT:D_DO-41_SOD81_P10.16mm_Horizontal" H 5750 3975 50  0001 C CNN
+F 2 "Diode_THT:D_DO-41_SOD81_P7.62mm_Horizontal" H 5750 3975 50  0001 C CNN
 F 3 "https://www.vishay.com/docs/85816/1n4728a.pdf" H 5750 4150 50  0001 C CNN
 	1    5750 4150
