File: Testing.kicad_pcb (KiCad board)
At the start: 2 copper layers, 60.5 x 25.9 mm, 18 parts, among them J4 Jack-DC, J6 In Sleeve, J7 Out Sleeve

Commit message: pcb layout: move some things around
This mostly involved swapping the transistor with the output coupling
capacitor so that the amplifier and feedback was on the left, and the
output stages were on the right.  I also rotated one resistor so the
nets were closer to each other, and swapped a few of the traces to other
layers of the PCB so that they could be shorter as well.

Overall, the result is pretty much just shorter traces and beefier
power-rail-fill in spots.
Parts:
- moved 10uF 31.2 mm to (195.3, 107.2)
- moved BS170 30.5 mm to (164.6, 106.9)
- moved R1 7.62 mm to (178.6, 103.4), turned to 270 degrees
Routing:
- net Net-(C2-Pad2): track 61.2 -> 12.0 mm
- net Net-(D1-Pad2): track 69.6 -> 28.0 mm
- net Net-(C1-Pad1): track 53.6 -> 32.6 mm
- net Net-(C2-Pad1): track 44.7 -> 35.4 mm
- net Net-(J5-Pad1): track 26.4 -> 28.4 mm
- net Net-(D2-Pad1): track 13.4 -> 14.2 mm
- net Net-(C1-Pad2): track 13.8 -> 14.5 mm
